File: ColorChangingGlucosePatch.kicad_sch (KiCad schematic)
At the start: 25 parts, among them U1 TPS76925DBVR, U2 TPS76925DBVR, U3 LMC6484, U7 CD4066BM96, U8 ATTINY204-SSFR

Commit message: final version but its not because im probably gonna work on it tomorrow.
Parts:
- C1, C2, C3, C4, C5, C6, C7, C8: footprint Capacitor_SMD:CP_Elec_3x5.3 -> Capacitor_SMD:C_0201_0603Metric_Pad0.64x0.40mm_HandSolder
- R1, R2, R4, R5: footprint Resistor_SMD:R_0201_0603Metric -> Capacitor_SMD:C_0201_0603Metric_Pad0.64x0.40mm_HandSolder
- R3: value R_US -> 100k; footprint Resistor_SMD:R_0201_0603Metric -> Capacitor_SMD:C_0201_0603Metric_Pad0.64x0.40mm_HandSolder
- R6, R7, R8: value R_US -> 180; footprint Resistor_SMD:R_0201_0603Metric -> Capacitor_SMD:C_0201_0603Metric_Pad0.64x0.40mm_HandSolder
- U3: footprint LMC6484AIN_NOPB-2:DIP254P762X508-14 -> LMC6484IMX_NOPB (1):SOIC127P600X175-14N
Connections:
- net +2.1V: now also U3.3 (+)
- net +2.5V: no longer U3.3 (+)
- net +5V: now also U8.1 (VDD)
- net GND: now also U8.14 (GND)
Changed lines of the file:
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@@
 	(wire
 		(pts
+			(xy 273.05 104.14) (xy 280.67 104.14)
+		)
+		(stroke
+			(width 0)
+			(type default)
+		)
+	)
+	(wire
+		(pts
+			(xy 212.09 99.06) (xy 212.09 104.14)
+		)
+		(stroke
+			(width 0)
+			(type default)
+		)
+	)
+	(wire
+		(pts
 			(xy 88.9 68.58) (xy 275.59 68.58)
 		)
@@
 			)
 		)
-		(property "Value" "R_US"
+		(property "Value" "180"
 			(at 275.59 147.3199 0)
 			(effects
@@
 			)
 		)
-		(property "Footprint" "Resistor_SMD:R_0201_0603Metric"
+		(property "Footprint" "Capacitor_SMD:C_0201_0603Metric_Pad0.64x0.40mm_HandSolder"
 			(at 274.066 146.304 90)
 			(effects
@@
 			)
 		)
-		(property "Footprint" "Capacitor_SMD:CP_Elec_3x5.3"
+		(property "Footprint" "Capacitor_SMD:C_0201_0603Metric_Pad0.64x0.40mm_HandSolder"
 			(at 96.52 95.5548 0)
 			(effects
@@
 			)
 		)
-		(property "Footprint" "LMC6484AIN_NOPB-2:DIP254P762X508-14"
+		(property "Footprint" "LMC6484IMX_NOPB (1):SOIC127P600X175-14N"
 			(at 30.48 33.02 0)
 			(effects
@@
 	(symbol
 		(lib_id "power:GND")
+		(at 280.67 104.14 0)
+		(unit 1)
+		(exclude_from_sim no)
+		(in_bom yes)
+		(on_board yes)
+		(dnp no)
+		(fields_autoplaced yes)
+		(property "Reference" "#PWR023"
+			(at 280.67 110.49 0)
+			(effects
+				(font
+					(size 1.27 1.27)
+				)
+				(hide yes)
+			)
+		)
+		(property "Value" "GND"
+			(at 280.67 109.22 0)
+			(effects
+				(font
+					(size 1.27 1.27)
+				)
+			)
+		)
+		(property "Footprint" ""
+			(at 280.67 104.14 0)
+			(effects
+				(font
+					(size 1.27 1.27)
+				)
+				(hide yes)
+			)
+		)
+		(property "Datasheet" ""
+			(at 280.67 104.14 0)
+			(effects
+				(font
+					(size 1.27 1.27)
+				)
+				(hide yes)
+			)
+		)
+		(property "Description" "Power symbol creates a global label with name \"GND\" , ground"
+			(at 280.67 104.14 0)
+			(effects
+				(font
+					(size 1.27 1.27)
+				)
+				(hide yes)
+			)
+		)
+		(pin "1"
+		)
+		(instances
+			(project ""
+				(path "/b5984cb0-ad73-4f98-955d-72ca9f838a44"
+					(reference "#PWR023")
+					(unit 1)
+				)
+			)
+		)
+	)
+	(symbol
+		(lib_id "power:GND")
 		(at 29.21 45.72 0)
 		(unit 1)
@@
 			)
 		)
-		(property "Value" "R_US"
+		(property "Value" "180"
 			(at 265.43 147.3199 0)
 			(effects
@@
 			)
 		)
-		(property "Footprint" "Resistor_SMD:R_0201_0603Metric"
+		(property "Footprint" "Capacitor_SMD:C_0201_0603Metric_Pad0.64x0.40mm_HandSolder"
 			(at 263.906 146.304 90)
 			(effects
@@
 			)
 		)
-		(property "Footprint" "LMC6484AIN_NOPB-2:DIP254P762X508-14"
+		(property "Footprint" "LMC6484IMX_NOPB (1):SOIC127P600X175-14N"
 			(at 78.74 133.35 0)
 			(effects
@@
 			)
 		)
-		(property "Value" "R_US"
+		(property "Value" "100k"
 			(at 72.39 116.84 90)
 			(effects
@@
 			)
 		)
-		(property "Footprint" "Resistor_SMD:R_0201_0603Metric"
+		(property "Footprint" "Capacitor_SMD:C_0201_0603Metric_Pad0.64x0.40mm_HandSolder"
 			(at 72.644 119.634 90)
 			(effects
@@
 			)
 		)
-		(property "Footprint" "Capacitor_SMD:CP_Elec_3x5.3"
+		(property "Footprint" "Capacitor_SMD:C_0201_0603Metric_Pad0.64x0.40mm_HandSolder"
 			(at 238.4552 38.1 0)
 			(effects
@@
 			)
 		)
-		(property "Value" "R_US"
+		(property "Value" "180"
 			(at 251.46 147.3199 0)
 			(effects
@@
 			)
 		)
-		(property "Footprint" "Resistor_SMD:R_0201_0603Metric"
+		(property "Footprint" "Capacitor_SMD:C_0201_0603Metric_Pad0.64x0.40mm_HandSolder"
 			(at 249.936 146.304 90)
 			(effects
@@
 			)
 		)
-		(property "Value" "+2.5V"
+		(property "Value" "+2.1V"
 			(at 20.32 25.4 0)
 			(effects
@@
 			)
 		)
-		(property "Footprint" "Capacitor_SMD:CP_Elec_3x5.3"
+		(property "Footprint" "Capacitor_SMD:C_0201_0603Metric_Pad0.64x0.40mm_HandSolder"
 			(at 163.5252 35.56 0)
 			(effects
@@
 			)
 		)
-		(property "Footprint" "Resistor_SMD:R_0201_0603Metric"
+		(property "Footprint" "Capacitor_SMD:C_0201_0603Metric_Pad0.64x0.40mm_HandSolder"
 			(at 163.576 56.134 90)
 			(effects
@@
 			)
 		)
-		(property "Footprint" "Capacitor_SMD:CP_Elec_3x5.3"
+		(property "Footprint" "Capacitor_SMD:C_0201_0603Metric_Pad0.64x0.40mm_HandSolder"
 			(at 185.1152 39.37 0)
 			(effects
@@
 			)
 		)
-		(property "Footprint" "Resistor_SMD:R_0201_0603Metric"
+		(property "Footprint" "Capacitor_SMD:C_0201_0603Metric_Pad0.64x0.40mm_HandSolder"
 			(at 54.864 105.664 90)
 			(effects
@@
 			)
 		)
-		(property "Footprint" "Resistor_SMD:R_0201_0603Metric"
+		(property "Footprint" "Capacitor_SMD:C_0201_0603Metric_Pad0.64x0.40mm_HandSolder"
 			(at 89.916 72.644 90)
 			(effects
@@
 			)
 		)
-		(property "Footprint" "Resistor_SMD:R_0201_0603Metric"
+		(property "Footprint" "Capacitor_SMD:C_0201_0603Metric_Pad0.64x0.40mm_HandSolder"
 			(at 163.576 44.704 90)
 			(effects
@@
 			)
 		)
-		(property "Footprint" "LMC6484AIN_NOPB-2:DIP254P762X508-14"
+		(property "Footprint" "LMC6484IMX_NOPB (1):SOIC127P600X175-14N"
 			(at 53.34 118.11 0)
 			(effects
@@
 			)
 		)
-		(property "Footprint" "Capacitor_SMD:CP_Elec_3x5.3"
+		(property "Footprint" "Capacitor_SMD:C_0201_0603Metric_Pad0.64x0.40mm_HandSolder"
 			(at 115.2652 35.56 0)
 			(effects
@@
 			)
 		)
-		(property "Footprint" "Capacitor_SMD:CP_Elec_3x5.3"
+		(property "Footprint" "Capacitor_SMD:C_0201_0603Metric_Pad0.64x0.40mm_HandSolder"
 			(at 43.18 25.7048 0)
 			(effects
@@
 			)
 		)
-		(property "Footprint" "Capacitor_SMD:CP_Elec_3x5.3"
+		(property "Footprint" "Capacitor_SMD:C_0201_0603Metric_Pad0.64x0.40mm_HandSolder"
 			(at 58.42 94.2848 0)
 			(effects
@@
 			)
 		)
-		(property "Footprint" "LMC6484AIN_NOPB-2:DIP254P762X508-14"
+		(property "Footprint" "LMC6484IMX_NOPB (1):SOIC127P600X175-14N"
 			(at 92.71 115.57 0)
 			(effects
@@
 			)
 		)
-		(property "Footprint" "Capacitor_SMD:CP_Elec_3x5.3"
+		(property "Footprint" "Capacitor_SMD:C_0201_0603Metric_Pad0.64x0.40mm_HandSolder"
 			(at 197.8152 139.7 0)
 			(effects
@@
 			)
 		)
-		(property "Footprint" "LMC6484AIN_NOPB-2:DIP254P762X508-14"
+		(property "Footprint" "LMC6484IMX_NOPB (1):SOIC127P600X175-14N"
 			(at 30.48 33.02 0)
 			(effects
@@
 					(unit 1)
 				)
+			)
+		)
+	)
+	(symbol
+		(lib_id "power:+5V")
+		(at 212.09 99.06 0)
+		(unit 1)
+		(exclude_from_sim no)
+		(in_bom yes)
+		(on_board yes)
+		(dnp no)
+		(fields_autoplaced yes)
+		(property "Reference" "#PWR022"
+			(at 212.09 102.87 0)
+			(effects
+				(font
+					(size 1.27 1.27)
+				)
+				(hide yes)
+			)
+		)
+		(property "Value" "+5V"
+			(at 212.09 93.98 0)
+			(effects
+				(font
+					(size 1.27 1.27)
+				)
+			)
+		)
+		(property "Footprint" ""
+			(at 212.09 99.06 0)
+			(effects
+				(font
+					(size 1.27 1.27)
+				)
+				(hide yes)
+			)
+		)
+		(property "Datasheet" ""
+			(at 212.09 99.06 0)
+			(effects
+				(font
+					(size 1.27 1.27)
+				)
+				(hide yes)
+			)
+		)
+		(property "Description" "Power symbol creates a global label with name \"+5V\""
+			(at 212.09 99.06 0)
+			(effects
+				(font
+					(size 1.27 1.27)
+				)
+				(hide yes)
+			)
+		)
+		(pin "1"
+		)
+		(instances
+			(project ""
+				(path "/b5984cb0-ad73-4f98-955d-72ca9f838a44"
+					(reference "#PWR022")
+					(unit 1)
+				)

Commit message: fuck this
Other:
- moved on the sheet: C8
Changed lines of the file:
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@@
 		(exclude_from_sim no)
 		(at 110.49 86.36 0)
-		(size 83.82 57.15)
+		(size 83.82 63.5)
 		(margins 0.9525 0.9525 0.9525 0.9525)
 		(stroke
@@
 	)
 	(junction
-		(at 196.85 129.54)
+		(at 191.77 129.54)
 		(diameter 0)
 		(color 0 0 0 0)
@@
 	(wire
 		(pts
-			(xy 196.85 129.54) (xy 196.85 128.27)
+			(xy 191.77 129.54) (xy 191.77 128.27)
 		)
 		(stroke
@@
 	(wire
 		(pts
-			(xy 196.85 129.54) (xy 196.85 132.08)
+			(xy 191.77 129.54) (xy 191.77 132.08)
 		)
 		(stroke
@@
 	(wire
 		(pts
-			(xy 196.85 139.7) (xy 196.85 143.51)
+			(xy 191.77 139.7) (xy 191.77 143.51)
 		)
 		(stroke
@@
 	(wire
 		(pts
-			(xy 185.42 129.54) (xy 196.85 129.54)
+			(xy 185.42 129.54) (xy 191.77 129.54)
 		)
 		(stroke
@@
 	(symbol
 		(lib_id "power:GND")
-		(at 196.85 143.51 0)
+		(at 191.77 143.51 0)
 		(unit 1)
 		(exclude_from_sim no)
@@
 		(fields_autoplaced yes)
 		(property "Reference" "#PWR016"
-			(at 196.85 149.86 0)
+			(at 191.77 149.86 0)
 			(effects
 				(font
@@
 		)
 		(property "Value" "GND"
-			(at 196.85 148.59 0)
+			(at 191.77 148.59 0)
 			(effects
 				(font
@@
 		)
 		(property "Footprint" ""
-			(at 196.85 143.51 0)
+			(at 191.77 143.51 0)
 			(effects
 				(font
@@
 		)
 		(property "Datasheet" ""
-			(at 196.85 143.51 0)
+			(at 191.77 143.51 0)
 			(effects
 				(font
@@
 		)
 		(property "Description" "Power symbol creates a global label with name \"GND\" , ground"
-			(at 196.85 143.51 0)
+			(at 191.77 143.51 0)
 			(effects
 				(font
@@
 	(symbol
 		(lib_id "power:+2.5V")
-		(at 196.85 128.27 0)
+		(at 191.77 128.27 0)
 		(unit 1)
 		(exclude_from_sim no)
@@
 		(fields_autoplaced yes)
 		(property "Reference" "#PWR015"
-			(at 196.85 132.08 0)
+			(at 191.77 132.08 0)
 			(effects
 				(font
@@
 		)
 		(property "Value" "+2.5V"
-			(at 196.85 123.19 0)
+			(at 191.77 123.19 0)
 			(effects
 				(font
@@
 		)
 		(property "Footprint" ""
-			(at 196.85 128.27 0)
+			(at 191.77 128.27 0)
 			(effects
 				(font
@@
 		)
 		(property "Datasheet" ""
-			(at 196.85 128.27 0)
+			(at 191.77 128.27 0)
 			(effects
 				(font
@@
 		)
 		(property "Description" "Power symbol creates a global label with name \"+5V\""
-			(at 196.85 128.27 0)
+			(at 191.77 128.27 0)
 			(effects
 				(font
@@
 	(symbol
 		(lib_id "Device:C")
-		(at 196.85 135.89 0)
+		(at 191.77 135.89 0)
 		(unit 1)
 		(exclude_from_sim no)
@@
 		(on_board yes)
 		(dnp no)
-		(fields_autoplaced yes)
 		(property "Reference" "C8"
-			(at 200.66 134.6199 0)
+			(at 184.15 134.62 0)
 			(effects
 				(font
@@
 		)
 		(property "Value" "100nF"
-			(at 200.66 137.1599 0)
+			(at 182.88 136.906 0)
 			(effects
 				(font
@@
 		)
 		(property "Footprint" "Capacitor_SMD:C_0201_0603Metric_Pad0.64x0.40mm_HandSolder"
-			(at 197.8152 139.7 0)
+			(at 192.7352 139.7 0)
 			(effects
 				(font
@@
 		)
 		(property "Datasheet" "~"
-			(at 196.85 135.89 0)
+			(at 191.77 135.89 0)
 			(effects
 				(font
@@
 		)
 		(property "Description" "Unpolarized capacitor"
-			(at 196.85 135.89 0)
+			(at 191.77 135.89 0)
 			(effects
 				(font
